Commit message: One robot shows up now

File: nuturtle_description/urdf/turtlebot3_burger.urdf.xacro (robot description, xacro)
@@ -46,5 +46,5 @@
       <origin xyz="-0.032 0 0.0" rpy="0 0 0"/>
       <geometry>
-        <mesh filename="package://nuturtle_description/burger_base.stl" scale="0.001 0.001 0.001"/>
+        <mesh filename="package://nuturtle_description/meshes/burger_base.stl" scale="0.001 0.001 0.001"/>
       </geometry>
       <material name="light_black"/>
@@ -72,5 +72,5 @@
       <origin xyz="0 0 0" rpy="1.57 0 0"/>
       <geometry>
-        <mesh filename="package://nuturtle_description/wheels/left_tire.stl" scale="0.001 0.001 0.001"/>
+        <mesh filename="package://nuturtle_description/meshes/left_tire.stl" scale="0.001 0.001 0.001"/>
       </geometry>
       <material name="dark"/>
@@ -98,5 +98,5 @@
       <origin xyz="0 0 0" rpy="1.57 0 0"/>
       <geometry>
-        <mesh filename="package://nuturtle_description/wheels/right_tire.stl" scale="0.001 0.001 0.001"/>
+        <mesh filename="package://nuturtle_description/meshes/right_tire.stl" scale="0.001 0.001 0.001"/>
       </geometry>
       <material name="dark"/>
@@ -147,5 +147,5 @@
       <origin xyz="0 0 0.0" rpy="0 0 0"/>
       <geometry>
-        <mesh filename="package://nuturtle_description/sensors/lds.stl" scale="0.001 0.001 0.001"/>
+        <mesh filename="package://nuturtle_description/meshes/lds.stl" scale="0.001 0.001 0.001"/>
       </geometry>
       <material name="dark"/>

Commit message: Task A.3

File: nuturtle_description/urdf/turtlebot3_burger.urdf.xacro (robot description, xacro)
@@ -3,4 +3,7 @@
   xmlns:xacro="http://ros.org/wiki/xacro">
 <!-- This file has been modified to replace all references to turtlebot3 files with copies made in this package -->
+  <xacro:property name="yaml" value="$(find nuturtle_description)/config/diff_params.yaml" />
+  <!-- Begin_Citation[2] -->
+  <xacro:property name="config" value="${xacro.load_yaml(yaml)['/**']['ros__parameters']}"/>
   <xacro:arg name="namespace" default=""/>
   <xacro:property name="namespace" value="$(arg namespace)"/>
@@ -53,5 +56,5 @@
       <origin xyz="-0.032 0 0.070" rpy="0 0 0"/>
       <geometry>
-        <box size="0.140 0.140 0.143"/>
+        <cylinder length=".0143" radius="${config['collision_radius']}"/>
       </geometry>
     </collision>
@@ -65,5 +68,5 @@
     <parent link="${namespace}base_link"/>
     <child link="${namespace}wheel_left_link"/>
-    <origin xyz="0.0 0.08 0.023" rpy="-1.57 0 0"/>
+    <origin xyz="0.0 ${config['track_width'] / 2} 0.023" rpy="-1.57 0 0"/>
     <axis xyz="0 0 1"/>
   </joint>
@@ -79,5 +82,5 @@
       <origin xyz="0 0 0" rpy="0 0 0"/>
       <geometry>
-        <cylinder length="0.018" radius="0.033"/>
+        <cylinder length="0.018" radius="${config['wheel_radius']}"/>
       </geometry>
     </collision>
@@ -91,5 +94,5 @@
     <parent link="${namespace}base_link"/>
     <child link="${namespace}wheel_right_link"/>
-    <origin xyz="0.0 -0.080 0.023" rpy="-1.57 0 0"/>
+    <origin xyz="0.0 ${-1 * config['track_width'] / 2} 0.023" rpy="-1.57 0 0"/>
     <axis xyz="0 0 1"/>
   </joint>
@@ -105,5 +108,5 @@
       <origin xyz="0 0 0" rpy="0 0 0"/>
       <geometry>
-        <cylinder length="0.018" radius="0.033"/>
+        <cylinder length="0.018" radius="${config['wheel_radius']}"/>
       </geometry>
     </collision>

Commit message: All of A

File: nuturtle_description/urdf/turtlebot3_burger.urdf.xacro (robot description, xacro)
@@ -6,6 +6,19 @@
   <!-- Begin_Citation[2] -->
   <xacro:property name="config" value="${xacro.load_yaml(yaml)['/**']['ros__parameters']}"/>
-  <xacro:arg name="namespace" default=""/>
-  <xacro:property name="namespace" value="$(arg namespace)"/>
+  <xacro:arg name="color" default=""/>
+  <xacro:property name="color" value="$(arg color)"/>
+  <xacro:if value="${color == 'red'}">
+    <xacro:property name="base_material" value="red"/>
+  </xacro:if>
+  <xacro:if value="${color == 'green'}">
+    <xacro:property name="base_material" value="green"/>
+  </xacro:if>
+  <xacro:if value="${color == 'blue'}">
+    <xacro:property name="base_material" value="blue"/>
+  </xacro:if>
+  <xacro:if value="${color == 'purple'}">
+    <xacro:property name="base_material" value="purple"/>
+  </xacro:if>
+  <xacro:property name="namespace" value=""/>
   <!-- Init colour -->
   <material name="black">
@@ -39,4 +52,7 @@
     <color rgba="1.0 1.0 1.0 1.0"/>
   </material>
+  <material name="purple">
+    <color rgba="0.3 .16 .52 1.0"/>
+  </material>
   <link name="${namespace}base_footprint"/>
   <joint name="${namespace}base_joint" type="fixed">
@@ -51,5 +67,5 @@
         <mesh filename="package://nuturtle_description/meshes/burger_base.stl" scale="0.001 0.001 0.001"/>
       </geometry>
-      <material name="light_black"/>
+      <material name="${base_material}"/>
     </visual>
     <collision>
@@ -77,5 +93,5 @@
         <mesh filename="package://nuturtle_description/meshes/left_tire.stl" scale="0.001 0.001 0.001"/>
       </geometry>
-      <material name="dark"/>
+      <material name="${base_material}"/>
     </visual>
     <collision>
@@ -103,5 +119,5 @@
         <mesh filename="package://nuturtle_description/meshes/right_tire.stl" scale="0.001 0.001 0.001"/>
       </geometry>
-      <material name="dark"/>
+      <material name="${base_material}"/>
     </visual>
     <collision>
@@ -152,5 +168,5 @@
         <mesh filename="package://nuturtle_description/meshes/lds.stl" scale="0.001 0.001 0.001"/>
       </geometry>
-      <material name="dark"/>
+      <material name="${base_material}"/>
     </visual>
     <collision>
